File: LightController/LightController.kicad_pcb (KiCad board)
At the start: 2 copper layers, 12 parts, among them Q1 BSS138, Q2 Q_NMOS_GDS, Q3 Q_NMOS_GDS, Q4 Q_NMOS_GDS, Q5 Q_NMOS_GDS, Q6 Q_NMOS_GDS, Q7 Q_NMOS_GDS, U1 ESP32-WROOM-32D, U2 AP3012

Commit message: Add footprints and shit.
Parts:
- added C1: C, Capacitor_SMD:C_1206_3216Metric, F.Cu at (81.8, 89.9)
- added C2: C, Capacitor_SMD:C_1206_3216Metric, F.Cu at (81.8, 93.2)
- added C3: C, Capacitor_SMD:C_1206_3216Metric, F.Cu at (81.8, 96.6)
- added C4: u1F, Capacitor_SMD:C_1206_3216Metric, F.Cu at (81.8, 99.9)
- added C5: 1uF, Capacitor_SMD:C_1206_3216Metric, F.Cu at (81.8, 103.3)
- added C6: u1F, Capacitor_SMD:C_1206_3216Metric, F.Cu at (81.8, 106.6)
- added C7: 1uF, Capacitor_SMD:C_1206_3216Metric, F.Cu at (81.8, 110.0)
- added C8: 10uF, Capacitor_SMD:C_1206_3216Metric, F.Cu at (81.8, 113.3)
- added C9: .1uF, Capacitor_SMD:C_1206_3216Metric, F.Cu at (81.8, 116.7)
- added D4: D, Diode_SMD:D_1206_3216Metric_Pad1.42x1.75mm_HandSolder, F.Cu at (93.3, 108.6)
- added D5: D, Diode_SMD:D_1206_3216Metric_Pad1.42x1.75mm_HandSolder, F.Cu at (93.3, 112.0)
- added J2: Conn_01x04, Connector_PinSocket_2.54mm:PinSocket_1x04_P2.54mm_Vertical, F.Cu at (87.0, 90.5)
- added J3: Conn_01x04, Connector_PinSocket_2.54mm:PinSocket_1x04_P2.54mm_Vertical, F.Cu at (91.6, 90.5)
- added R11: 110ohm, Resistor_SMD:R_1206_3216Metric, F.Cu at (87.5, 102.1)
- added R12: 330ohm, Resistor_SMD:R_1206_3216Metric, F.Cu at (87.5, 105.4)
- added R13: 330 ohm, Resistor_SMD:R_1206_3216Metric, F.Cu at (87.5, 108.7)
- added R14: 200 ohm, Resistor_SMD:R_1206_3216Metric, F.Cu at (87.5, 112.0)
- added U3: AP3012, Package_TO_SOT_SMD:SOT-23-5, F.Cu at (92.8, 115.9)
- added U4: MAX485E, Package_SO:SOP-8_3.9x4.9mm_P1.27mm, F.Cu at (94.5, 103.7)
Connections:
- Q2 pad 2: unconnected-(Q2-D) -> Net-(J2-Pin_2)
- Q2 pad 3: unconnected-(Q2-S) -> GND
- Q3 pad 2: unconnected-(Q3-D) -> Net-(J2-Pin_3)
- Q3 pad 3: unconnected-(Q3-S) -> GND
- Q4 pad 2: unconnected-(Q4-D) -> Net-(J2-Pin_4)
- Q4 pad 3: unconnected-(Q4-S) -> GND
- Q5 pad 2: unconnected-(Q5-D) -> Net-(J3-Pin_2)
- Q5 pad 3: unconnected-(Q5-S) -> GND
- Q6 pad 2: unconnected-(Q6-D) -> Net-(J3-Pin_3)
- Q6 pad 3: unconnected-(Q6-S) -> GND
- Q7 pad 2: unconnected-(Q7-D) -> Net-(J3-Pin_4)
- Q7 pad 3: unconnected-(Q7-S) -> GND
