File: TeamSign/TeamSign.kicad_pcb (KiCad board)
At the start: 2 copper layers, 259.2 x 139.8 mm, 105 parts, among them J1 RJ45, J2 Barrel_Jack_MountingPin, U1 TPS563200, U2 ESP32-Devkit_C_V4

Commit message: Shrink the labels for the side-firing SK6812SideAs, as well as start the footprint of the SMTSOM2.550BTR PEM nut.
Other:
- board size 259.2 x 139.8 mm -> 241.2 x 139.8 mm
Changed lines of the file:
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@@
     (property "ki_keywords" "SK6812 \"NeoPixel\" Style LED, with side-firing orientation and discrete pinout.")
     (attr smd)
-    (fp_text reference "D30" (at -9.75 -15.85 90 unlocked) (layer "F.SilkS")
+    (fp_text reference "D30" (at -0.2764 -2.5379 90 unlocked) (layer "F.SilkS")
         (effects (font (size 1 1) (thickness 0.1)))
     )
-    (fp_text value "SK6812-Side-A" (at -9.75 -14.35 90 unlocked) (layer "F.Fab")
+    (fp_text value "SK6812-Side-A" (at -0.3404 -3.9029 90 unlocked) (layer "F.Fab")
         (effects (font (size 1 1) (thickness 0.15)))
     )
-    (fp_text user "${REFERENCE}" (at -9.75 -12.85 90 unlocked) (layer "F.Fab")
+    (fp_text user "${REFERENCE}" (at -0.3404 -2.4029 90 unlocked) (layer "F.Fab")
         (effects (font (size 1 1) (thickness 0.15)))
     )
@@
     (property "ki_keywords" "SK6812 \"NeoPixel\" Style LED, with side-firing orientation and discrete pinout.")
     (attr smd)
-    (fp_text reference "D29" (at -9.75 -15.85 90 unlocked) (layer "F.SilkS")
+    (fp_text reference "D29" (at -0.3404 -5.4029 90 unlocked) (layer "F.SilkS")
         (effects (font (size 1 1) (thickness 0.1)))
     )
-    (fp_text value "SK6812-Side-A" (at -9.75 -14.35 90 unlocked) (layer "F.Fab")
+    (fp_text value "SK6812-Side-A" (at -0.3404 -3.9029 90 unlocked) (layer "F.Fab")
         (effects (font (size 1 1) (thickness 0.15)))
     )
-    (fp_text user "${REFERENCE}" (at -9.75 -12.85 90 unlocked) (layer "F.Fab")
+    (fp_text user "${REFERENCE}" (at -0.3404 -2.4029 90 unlocked) (layer "F.Fab")
         (effects (font (size 1 1) (thickness 0.15)))
     )
@@
     (property "ki_keywords" "SK6812 \"NeoPixel\" Style LED, with side-firing orientation and discrete pinout.")
     (attr smd)
-    (fp_text reference "D31" (at -9.75 -15.85 90 unlocked) (layer "F.SilkS")
+    (fp_text reference "D31" (at -0.1104 -2.1489 90 unlocked) (layer "F.SilkS")
         (effects (font (size 1 1) (thickness 0.1)))
     )
-    (fp_text value "SK6812-Side-A" (at -9.75 -14.35 90 unlocked) (layer "F.Fab")
+    (fp_text value "SK6812-Side-A" (at -0.3404 -3.9029 90 unlocked) (layer "F.Fab")
         (effects (font (size 1 1) (thickness 0.15)))
     )
-    (fp_text user "${REFERENCE}" (at -9.75 -12.85 90 unlocked) (layer "F.Fab")
+    (fp_text user "${REFERENCE}" (at -0.3404 -2.4029 90 unlocked) (layer "F.Fab")
         (effects (font (size 1 1) (thickness 0.15)))
     )
@@
     (property "ki_keywords" "SK6812 \"NeoPixel\" Style LED, with side-firing orientation and discrete pinout.")
     (attr smd)
-    (fp_text reference "D32" (at -9.75 -15.85 90 unlocked) (layer "F.SilkS")
+    (fp_text reference "D32" (at -0.3404 -2.7719 90 unlocked) (layer "F.SilkS")
         (effects (font (size 1 1) (thickness 0.1)))
     )
-    (fp_text value "SK6812-Side-A" (at -9.75 -14.35 90 unlocked) (layer "F.Fab")
+    (fp_text value "SK6812-Side-A" (at -0.3404 -3.9029 90 unlocked) (layer "F.Fab")
         (effects (font (size 1 1) (thickness 0.15)))
     )
-    (fp_text user "${REFERENCE}" (at -9.75 -12.85 90 unlocked) (layer "F.Fab")
+    (fp_text user "${REFERENCE}" (at -0.3404 -2.4029 90 unlocked) (layer "F.Fab")
         (effects (font (size 1 1) (thickness 0.15)))
     )
@@
     (property "ki_keywords" "SK6812 \"NeoPixel\" Style LED, with side-firing orientation and discrete pinout.")
     (attr smd)
-    (fp_text reference "D26" (at -9.75 -15.85 90 unlocked) (layer "F.SilkS")
+    (fp_text reference "D26" (at -0.3404 -5.4029 90 unlocked) (layer "F.SilkS")
         (effects (font (size 1 1) (thickness 0.1)))
     )
-    (fp_text value "SK6812-Side-A" (at -9.75 -14.35 90 unlocked) (layer "F.Fab")
+    (fp_text value "SK6812-Side-A" (at -0.3404 -3.9029 90 unlocked) (layer "F.Fab")
         (effects (font (size 1 1) (thickness 0.15)))
     )
-    (fp_text user "${REFERENCE}" (at -9.75 -12.85 90 unlocked) (layer "F.Fab")
+    (fp_text user "${REFERENCE}" (at -0.3404 -2.4029 90 unlocked) (layer "F.Fab")
         (effects (font (size 1 1) (thickness 0.15)))
     )
@@
     (property "ki_keywords" "SK6812 \"NeoPixel\" Style LED, with side-firing orientation and discrete pinout.")
     (attr smd)
-    (fp_text reference "D28" (at -9.75 -15.85 90 unlocked) (layer "F.SilkS")
+    (fp_text reference "D28" (at -0.3404 -5.4029 90 unlocked) (layer "F.SilkS")
         (effects (font (size 1 1) (thickness 0.1)))
     )
-    (fp_text value "SK6812-Side-A" (at -9.75 -14.35 90 unlocked) (layer "F.Fab")
+    (fp_text value "SK6812-Side-A" (at -0.3404 -3.9029 90 unlocked) (layer "F.Fab")
         (effects (font (size 1 1) (thickness 0.15)))
     )
-    (fp_text user "${REFERENCE}" (at -9.75 -12.85 90 unlocked) (layer "F.Fab")
+    (fp_text user "${REFERENCE}" (at -0.3404 -2.4029 90 unlocked) (layer "F.Fab")
         (effects (font (size 1 1) (thickness 0.15)))
     )
@@
     (property "ki_keywords" "SK6812 \"NeoPixel\" Style LED, with side-firing orientation and discrete pinout.")
     (attr smd)
-    (fp_text reference "D33" (at -9.75 -15.85 90 unlocked) (layer "F.SilkS")
+    (fp_text reference "D33" (at -0.3404 -2.6529 90 unlocked) (layer "F.SilkS")
         (effects (font (size 1 1) (thickness 0.1)))
     )
-    (fp_text value "SK6812-Side-A" (at -9.75 -14.35 90 unlocked) (layer "F.Fab")
+    (fp_text value "SK6812-Side-A" (at -0.3404 -3.9029 90 unlocked) (layer "F.Fab")
         (effects (font (size 1 1) (thickness 0.15)))
     )
-    (fp_text user "${REFERENCE}" (at -9.75 -12.85 90 unlocked) (layer "F.Fab")
+    (fp_text user "${REFERENCE}" (at -0.3404 -2.4029 90 unlocked) (layer "F.Fab")
         (effects (font (size 1 1) (thickness 0.15)))
     )
@@
     (property "ki_keywords" "SK6812 \"NeoPixel\" Style LED, with side-firing orientation and discrete pinout.")
     (attr smd)
-    (fp_text reference "D27" (at -9.75 -15.85 90 unlocked) (layer "F.SilkS")
+    (fp_text reference "D27" (at -0.3404 -5.4029 90 unlocked) (layer "F.SilkS")
         (effects (font (size 1 1) (thickness 0.1)))
     )
-    (fp_text value "SK6812-Side-A" (at -9.75 -14.35 90 unlocked) (layer "F.Fab")
+    (fp_text value "SK6812-Side-A" (at -0.3404 -3.9029 90 unlocked) (layer "F.Fab")
         (effects (font (size 1 1) (thickness 0.15)))
     )
-    (fp_text user "${REFERENCE}" (at -9.75 -12.85 90 unlocked) (layer "F.Fab")
+    (fp_text user "${REFERENCE}" (at -0.3404 -2.4029 90 unlocked) (layer "F.Fab")
         (effects (font (size 1 1) (thickness 0.15)))
     )
@@
       (net 1 "GND") (pintype "passive"))
   )
-  (gr_rect (start 14 19.25) (end 273.25 159)
+  (gr_rect (start 32 19.25) (end 273.25 159)
     (stroke (width 0.1) (type default)) (fill none) (layer "Edge.Cuts"))
   (gr_text "888" (at 30.9499 162.5346) (layer "F.SilkS")

Commit message: Place caps :)
Parts:
- removed C1, C97: 10uF, Capacitor_SMD:C_1206_3216Metric_Pad1.33x1.80mm_HandSolder
- removed C2: 100nF, Capacitor_SMD:C_1206_3216Metric_Pad1.33x1.80mm_HandSolder
- removed C3, C96: 22uF, Capacitor_SMD:CP_Elec_5x5.4
- removed D26, D27, D28, D29, D30, D31, D32, D33: SK6812-Side-A, footprints:SK6812-Side-A
- added C10: 100nF, Capacitor_SMD:C_1206_3216Metric_Pad1.33x1.80mm_HandSolder, F.Cu at (253.0, 70.4)
- added C11: 100nF, Capacitor_SMD:C_1206_3216Metric_Pad1.33x1.80mm_HandSolder, F.Cu at (80.8, 62.5)
- added C12: 100nF, Capacitor_SMD:C_1206_3216Metric_Pad1.33x1.80mm_HandSolder, F.Cu at (130.5, 87.7)
- added C13: 100nF, Capacitor_SMD:C_1206_3216Metric_Pad1.33x1.80mm_HandSolder, F.Cu at (252.0, 115.3)
- added C14: 100nF, Capacitor_SMD:C_1206_3216Metric_Pad1.33x1.80mm_HandSolder, F.Cu at (91.2, 66.8)
- added C15: 100nF, Capacitor_SMD:C_1206_3216Metric_Pad1.33x1.80mm_HandSolder, F.Cu at (141.3, 96.0)
- added C16: 100nF, Capacitor_SMD:C_1206_3216Metric_Pad1.33x1.80mm_HandSolder, F.Cu at (219.6, 139.8)
- added C17: 100nF, Capacitor_SMD:C_1206_3216Metric_Pad1.33x1.80mm_HandSolder, F.Cu at (91.0, 73.2)
- added C18: 100nF, Capacitor_SMD:C_1206_3216Metric_Pad1.33x1.80mm_HandSolder, F.Cu at (171.8, 133.2)
- added C19: 100nF, Capacitor_SMD:C_1206_3216Metric_Pad1.33x1.80mm_HandSolder, F.Cu at (211.8, 133.5)
- added C20: 100nF, Capacitor_SMD:C_1206_3216Metric_Pad1.33x1.80mm_HandSolder, F.Cu at (91.0, 79.5)
- added C21: 100nF, Capacitor_SMD:C_1206_3216Metric_Pad1.33x1.80mm_HandSolder, F.Cu at (141.5, 140.0)
- added C22: 100nF, Capacitor_SMD:C_1206_3216Metric_Pad1.33x1.80mm_HandSolder, F.Cu at (211.2, 86.9)
- added C23: 100nF, Capacitor_SMD:C_1206_3216Metric_Pad1.33x1.80mm_HandSolder, F.Cu at (91.2, 87.0)
- added C24: 100nF, Capacitor_SMD:C_1206_3216Metric_Pad1.33x1.80mm_HandSolder, F.Cu at (130.2, 133.9)
- added C25: 100nF, Capacitor_SMD:C_1206_3216Metric_Pad1.33x1.80mm_HandSolder, F.Cu at (221.5, 95.5)
- added C26: 100nF, Capacitor_SMD:C_1206_3216Metric_Pad1.33x1.80mm_HandSolder, F.Cu at (91.2, 112.2)
- added C27: 100nF, Capacitor_SMD:C_1206_3216Metric_Pad1.33x1.80mm_HandSolder, F.Cu at (146.0, 60.8)
- added C28: 100nF, Capacitor_SMD:C_1206_3216Metric_Pad1.33x1.80mm_HandSolder, F.Cu at (226.3, 60.8)
- added C29: 100nF, Capacitor_SMD:C_1206_3216Metric_Pad1.33x1.80mm_HandSolder, F.Cu at (0.40, 127.3)
- added C30: 100nF, Capacitor_SMD:C_1206_3216Metric_Pad1.33x1.80mm_HandSolder, F.Cu at (0.28, 124.1)
- added C31: 100nF, Capacitor_SMD:C_1206_3216Metric_Pad1.33x1.80mm_HandSolder, F.Cu at (0.40, 117.8)
- added C32: 100nF, Capacitor_SMD:C_1206_3216Metric_Pad1.33x1.80mm_HandSolder, F.Cu at (0.40, 121.2)
- added C33: 100nF, Capacitor_SMD:C_1206_3216Metric_Pad1.33x1.80mm_HandSolder, F.Cu at (6.59, 117.3)
- added C34: 100nF, Capacitor_SMD:C_1206_3216Metric_Pad1.33x1.80mm_HandSolder, F.Cu at (6.59, 120.7)
- added C35: 100nF, Capacitor_SMD:C_1206_3216Metric_Pad1.33x1.80mm_HandSolder, F.Cu at (6.59, 124.0)
- added C36: 100nF, Capacitor_SMD:C_1206_3216Metric_Pad1.33x1.80mm_HandSolder, F.Cu at (6.59, 127.4)
- added C37: 100nF, Capacitor_SMD:C_1206_3216Metric_Pad1.33x1.80mm_HandSolder, F.Cu at (91.2, 119.0)
- added C38: 100nF, Capacitor_SMD:C_1206_3216Metric_Pad1.33x1.80mm_HandSolder, F.Cu at (172.2, 75.3)
- added C39: 100nF, Capacitor_SMD:C_1206_3216Metric_Pad1.33x1.80mm_HandSolder, F.Cu at (253.0, 76.4)
- added C4: 100nF, Capacitor_SMD:C_1206_3216Metric_Pad1.33x1.80mm_HandSolder, F.Cu at (67.5, 62.8)
- added C40: 100nF, Capacitor_SMD:C_1206_3216Metric_Pad1.33x1.80mm_HandSolder, F.Cu at (91.2, 125.5)
- added C41: 100nF, Capacitor_SMD:C_1206_3216Metric_Pad1.33x1.80mm_HandSolder, F.Cu at (130.5, 81.7)
- added C42: 100nF, Capacitor_SMD:C_1206_3216Metric_Pad1.33x1.80mm_HandSolder, F.Cu at (147.3, 96.0)
- added C43: 100nF, Capacitor_SMD:C_1206_3216Metric_Pad1.33x1.80mm_HandSolder, F.Cu at (252.0, 121.3)
- added C44: 100nF, Capacitor_SMD:C_1206_3216Metric_Pad1.33x1.80mm_HandSolder, F.Cu at (91.2, 132.0)
- added C45: 100nF, Capacitor_SMD:C_1206_3216Metric_Pad1.33x1.80mm_HandSolder, F.Cu at (171.8, 127.2)
- added C46: 100nF, Capacitor_SMD:C_1206_3216Metric_Pad1.33x1.80mm_HandSolder, F.Cu at (225.6, 139.8)
- added C47: 100nF, Capacitor_SMD:C_1206_3216Metric_Pad1.33x1.80mm_HandSolder, F.Cu at (59.2, 95.0)
- added C48: 100nF, Capacitor_SMD:C_1206_3216Metric_Pad1.33x1.80mm_HandSolder, F.Cu at (147.5, 140.0)
- added C49: 100nF, Capacitor_SMD:C_1206_3216Metric_Pad1.33x1.80mm_HandSolder, F.Cu at (211.8, 127.5)
- added C5: 100nF, Capacitor_SMD:C_1206_3216Metric_Pad1.33x1.80mm_HandSolder, F.Cu at (61.5, 62.8)
- added C50: 100nF, Capacitor_SMD:C_1206_3216Metric_Pad1.33x1.80mm_HandSolder, F.Cu at (51.2, 88.0)
- added C51: 100nF, Capacitor_SMD:C_1206_3216Metric_Pad1.33x1.80mm_HandSolder, F.Cu at (130.2, 127.9)
- added C52: 100nF, Capacitor_SMD:C_1206_3216Metric_Pad1.33x1.80mm_HandSolder, F.Cu at (211.2, 80.9)
- added C53: 100nF, Capacitor_SMD:C_1206_3216Metric_Pad1.33x1.80mm_HandSolder, F.Cu at (51.2, 81.2)
- added C54: 100nF, Capacitor_SMD:C_1206_3216Metric_Pad1.33x1.80mm_HandSolder, F.Cu at (152.0, 60.8)
- added C55: 100nF, Capacitor_SMD:C_1206_3216Metric_Pad1.33x1.80mm_HandSolder, F.Cu at (227.5, 95.5)
- added C56: 100nF, Capacitor_SMD:C_1206_3216Metric_Pad1.33x1.80mm_HandSolder, F.Cu at (51.5, 74.5)
- added C57: 100nF, Capacitor_SMD:C_1206_3216Metric_Pad1.33x1.80mm_HandSolder, F.Cu at (172.2, 81.3)
- added C58: 100nF, Capacitor_SMD:C_1206_3216Metric_Pad1.33x1.80mm_HandSolder, F.Cu at (232.3, 60.8)
- added C59: 100nF, Capacitor_SMD:C_1206_3216Metric_Pad1.33x1.80mm_HandSolder, F.Cu at (52.0, 68.8)
- added C6: 100nF, Capacitor_SMD:C_1206_3216Metric_Pad1.33x1.80mm_HandSolder, F.Cu at (140.0, 60.8)
- added C60: 100nF, Capacitor_SMD:C_1206_3216Metric_Pad1.33x1.80mm_HandSolder, F.Cu at (130.5, 75.7)
- added C61: 100nF, Capacitor_SMD:C_1206_3216Metric_Pad1.33x1.80mm_HandSolder, F.Cu at (253.0, 82.4)
- added C62: 100nF, Capacitor_SMD:C_1206_3216Metric_Pad1.33x1.80mm_HandSolder, F.Cu at (51.2, 131.2)
- added C63: 100nF, Capacitor_SMD:C_1206_3216Metric_Pad1.33x1.80mm_HandSolder, F.Cu at (153.3, 96.0)
- added C64: 100nF, Capacitor_SMD:C_1206_3216Metric_Pad1.33x1.80mm_HandSolder, F.Cu at (252.0, 127.3)
- added C65: 100nF, Capacitor_SMD:C_1206_3216Metric_Pad1.33x1.80mm_HandSolder, F.Cu at (51.2, 124.8)
- added C66: 100nF, Capacitor_SMD:C_1206_3216Metric_Pad1.33x1.80mm_HandSolder, F.Cu at (171.8, 121.2)
- added C67: 100nF, Capacitor_SMD:C_1206_3216Metric_Pad1.33x1.80mm_HandSolder, F.Cu at (231.6, 139.8)
- added C68: 100nF, Capacitor_SMD:C_1206_3216Metric_Pad1.33x1.80mm_HandSolder, F.Cu at (51.2, 118.2)
- added C69: 100nF, Capacitor_SMD:C_1206_3216Metric_Pad1.33x1.80mm_HandSolder, F.Cu at (153.5, 140.0)
- added C7: 100nF, Capacitor_SMD:C_1206_3216Metric_Pad1.33x1.80mm_HandSolder, F.Cu at (220.3, 60.8)
- added C70: 100nF, Capacitor_SMD:C_1206_3216Metric_Pad1.33x1.80mm_HandSolder, F.Cu at (211.8, 121.5)
- added C71: 100nF, Capacitor_SMD:C_1206_3216Metric_Pad1.33x1.80mm_HandSolder, F.Cu at (211.2, 74.9)
- added C72: 100nF, Capacitor_SMD:C_1206_3216Metric_Pad1.33x1.80mm_HandSolder, F.Cu at (51.2, 111.8)
- added C73: 100nF, Capacitor_SMD:C_1206_3216Metric_Pad1.33x1.80mm_HandSolder, F.Cu at (130.2, 121.9)
- added C74: 100nF, Capacitor_SMD:C_1206_3216Metric_Pad1.33x1.80mm_HandSolder, F.Cu at (233.5, 95.5)
- added C75: 100nF, Capacitor_SMD:C_1206_3216Metric_Pad1.33x1.80mm_HandSolder, F.Cu at (57.5, 138.8)
- added C76: 100nF, Capacitor_SMD:C_1206_3216Metric_Pad1.33x1.80mm_HandSolder, F.Cu at (158.0, 60.8)
- added C77: 100nF, Capacitor_SMD:C_1206_3216Metric_Pad1.33x1.80mm_HandSolder, F.Cu at (238.3, 60.8)
- added C78: 100nF, Capacitor_SMD:C_1206_3216Metric_Pad1.33x1.80mm_HandSolder, F.Cu at (64.6, 138.8)
- added C79: 100nF, Capacitor_SMD:C_1206_3216Metric_Pad1.33x1.80mm_HandSolder, F.Cu at (172.2, 87.3)
- added C799: 100nF, Capacitor_SMD:C_1206_3216Metric_Pad1.33x1.80mm_HandSolder, F.Cu at (148.5, 37.8)
- added C8: 100nF, Capacitor_SMD:C_1206_3216Metric_Pad1.33x1.80mm_HandSolder, F.Cu at (74.0, 62.8)
- added C80: 100nF, Capacitor_SMD:C_1206_3216Metric_Pad1.33x1.80mm_HandSolder, F.Cu at (253.0, 88.4)
- added C81: 100nF, Capacitor_SMD:C_1206_3216Metric_Pad1.33x1.80mm_HandSolder, F.Cu at (72.0, 139.2)
- added C82: 100nF, Capacitor_SMD:C_1206_3216Metric_Pad1.33x1.80mm_HandSolder, F.Cu at (130.5, 69.7)
- added C83: 100nF, Capacitor_SMD:C_1206_3216Metric_Pad1.33x1.80mm_HandSolder, F.Cu at (252.0, 133.3)
- added C84: 100nF, Capacitor_SMD:C_1206_3216Metric_Pad1.33x1.80mm_HandSolder, F.Cu at (78.2, 139.0)
- added C85: 100nF, Capacitor_SMD:C_1206_3216Metric_Pad1.33x1.80mm_HandSolder, F.Cu at (159.3, 96.0)
- added C86: 100nF, Capacitor_SMD:C_1206_3216Metric_Pad1.33x1.80mm_HandSolder, F.Cu at (237.6, 139.8)
- added C87: 100nF, Capacitor_SMD:C_1206_3216Metric_Pad1.33x1.80mm_HandSolder, F.Cu at (79.0, 95.0)
- added C88: 100nF, Capacitor_SMD:C_1206_3216Metric_Pad1.33x1.80mm_HandSolder, F.Cu at (171.7, 115.2)
- added C89: 100nF, Capacitor_SMD:C_1206_3216Metric_Pad1.33x1.80mm_HandSolder, F.Cu at (211.8, 115.5)
- added C898: 22uF, Capacitor_SMD:CP_Elec_5x5.4, F.Cu at (168.2, 26.2)
- added C899: 22uF, Capacitor_SMD:CP_Elec_5x5.4, F.Cu at (168.2, 33.1)
- added C9: 100nF, Capacitor_SMD:C_1206_3216Metric_Pad1.33x1.80mm_HandSolder, F.Cu at (172.2, 69.3)
- added C90: 100nF, Capacitor_SMD:C_1206_3216Metric_Pad1.33x1.80mm_HandSolder, F.Cu at (72.0, 95.0)
- added C91: 100nF, Capacitor_SMD:C_1206_3216Metric_Pad1.33x1.80mm_HandSolder, F.Cu at (159.5, 140.0)
- added C92: 100nF, Capacitor_SMD:C_1206_3216Metric_Pad1.33x1.80mm_HandSolder, F.Cu at (211.2, 68.9)
- added C93: 100nF, Capacitor_SMD:C_1206_3216Metric_Pad1.33x1.80mm_HandSolder, F.Cu at (65.8, 95.0)
- added C94: 100nF, Capacitor_SMD:C_1206_3216Metric_Pad1.33x1.80mm_HandSolder, F.Cu at (130.2, 115.9)
- added C95: 100nF, Capacitor_SMD:C_1206_3216Metric_Pad1.33x1.80mm_HandSolder, F.Cu at (239.5, 95.5)
- added C998: 10uF, Capacitor_SMD:C_1206_3216Metric_Pad1.33x1.80mm_HandSolder, F.Cu at (160.6, 36.2)
- added C999: 10uF, Capacitor_SMD:C_1206_3216Metric_Pad1.33x1.80mm_HandSolder, F.Cu at (160.6, 39.6)
- added D300: SK6812-Side-A, footprints:SK6812-Side-A, F.Cu at (-5.67, 110.9)
- added D301: SK6812-Side-A, footprints:SK6812-Side-A, F.Cu at (-5.67, 113.9)
- added D302: SK6812-Side-A, footprints:SK6812-Side-A, F.Cu at (-5.67, 116.8)
- added D303: SK6812-Side-A, footprints:SK6812-Side-A, F.Cu at (-5.67, 119.8)
- added D304: SK6812-Side-A, footprints:SK6812-Side-A, F.Cu at (-5.67, 122.7)
- added D305: SK6812-Side-A, footprints:SK6812-Side-A, F.Cu at (-5.67, 125.7)
- added D306: SK6812-Side-A, footprints:SK6812-Side-A, F.Cu at (-5.67, 128.6)
- added D307: SK6812-Side-A, footprints:SK6812-Side-A, F.Cu at (-5.67, 131.6)

Commit message: Added gerbers for TS to the ignore, plus added level shifting.  Yay!
Parts:
- added Q1: BSS138, Package_TO_SOT_SMD:SOT-23, F.Cu at (213.1, 29.8)
- added Q2: BSS138, Package_TO_SOT_SMD:SOT-23, F.Cu at (213.1, 34.2)
- added R4: 10kΩ, Resistor_SMD:R_0805_2012Metric_Pad1.20x1.40mm_HandSolder, F.Cu at (213.0, 17.2)
- added R5: 10kΩ, Resistor_SMD:R_0805_2012Metric_Pad1.20x1.40mm_HandSolder, F.Cu at (213.0, 20.2)
- added R6: 10kΩ, Resistor_SMD:R_0805_2012Metric_Pad1.20x1.40mm_HandSolder, F.Cu at (213.0, 23.1)
- added R7: 10kΩ, Resistor_SMD:R_0805_2012Metric_Pad1.20x1.40mm_HandSolder, F.Cu at (213.0, 26.1)
- moved D300 233.1 mm to (207.7, 16.9)
- moved D301 233.1 mm to (207.7, 19.9)
- moved D302 233.1 mm to (207.7, 22.8)
- moved D303 233.1 mm to (207.7, 25.8)
- moved D304 233.1 mm to (207.7, 28.8)
- moved D305 233.1 mm to (207.7, 31.7)
- moved D306 233.1 mm to (207.7, 34.7)
- moved D307 233.1 mm to (207.7, 37.6)
- moved C29 229.4 mm to (201.7, 17.4)
- moved C30 226.4 mm to (201.7, 20.8)
- moved C31 222.1 mm to (201.7, 24.1)
- moved C32 222.1 mm to (201.7, 27.5)
- moved C33 213.5 mm to (201.7, 30.9)
- moved C34 213.5 mm to (201.7, 34.2)
- moved C35 213.5 mm to (201.7, 37.5)
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Connections:
- D1 pad 2: /sk_input -> /sk_lvl_shifted
- D300 pad 1: /stacklight_out -> /stacklight_lvl_shift
- U2 pad 20: unconnected-(U2-3.3v-Pad20) -> +3.3V
Routing:
- net GND: track 0.00 -> 1712.3 mm, vias 0 -> 5
- net +3V3: track 0.00 -> 1078.1 mm, vias 0 -> 18
- net +5V: track 0.00 -> 981.3 mm, vias 0 -> 17
- net /LED Array 1/sk_output_pin: track 0.00 -> 111.6 mm, vias 0 -> 2
- net +12V: track 0.00 -> 99.9 mm
- net /LED Array 2/sk_output_pin: track 0.00 -> 72.7 mm, vias 0 -> 2
- net Net-(D20-DOUT): track 0.00 -> 71.2 mm, vias 0 -> 2
- net /LED Array 3/sk_pin1: track 0.00 -> 68.8 mm, vias 0 -> 2
- net /LED Array 2/sk_pin2: track 0.00 -> 61.0 mm, vias 0 -> 2
- net Net-(D51-DOUT): track 0.00 -> 60.0 mm, vias 0 -> 2
- net /LED Array 3/sk_pin2: track 0.00 -> 58.8 mm, vias 0 -> 2
- net /LED Array 2/sk_pin1: track 0.00 -> 57.6 mm, vias 0 -> 2
- net Net-(U1-VFB): track 0.00 -> 50.5 mm, vias 0 -> 2
- net Net-(D16-DOUT): track 0.00 -> 48.2 mm
- net Net-(D88-DOUT): track 0.00 -> 48.1 mm, vias 0 -> 4
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- added copper zone on F.Cu, net GND

Commit message: Resolve subsheet antics... Yay.
Parts:
- removed C87, C90, C93: 100nF, Capacitor_SMD:C_1206_3216Metric_Pad1.33x1.80mm_HandSolder
- removed D34, D35, D36: SK6812, LED_SMD:LED_SK6812_PLCC4_5.0x5.0mm_P3.2mm
- added C1: 100nF, Capacitor_SMD:C_1206_3216Metric_Pad1.33x1.80mm_HandSolder, F.Cu at (79.0, 65.5)
- added C2: 100nF, Capacitor_SMD:C_1206_3216Metric_Pad1.33x1.80mm_HandSolder, F.Cu at (79.0, 68.8)
- added C3: 100nF, Capacitor_SMD:C_1206_3216Metric_Pad1.33x1.80mm_HandSolder, F.Cu at (79.0, 72.2)
- added D26: SK6812, LED_SMD:LED_SK6812_PLCC4_5.0x5.0mm_P3.2mm, F.Cu at (71.8, 93.6)
- added D27: SK6812, LED_SMD:LED_SK6812_PLCC4_5.0x5.0mm_P3.2mm, F.Cu at (71.8, 100.2)
- added D28: SK6812, LED_SMD:LED_SK6812_PLCC4_5.0x5.0mm_P3.2mm, F.Cu at (71.8, 106.9)
- moved D15 77.3 mm to (63.4, 67.1), turned to 0 degrees
- moved C65 74.9 mm to (97.0, 65.5), turned to 0 degrees
- moved C75 74.5 mm to (97.0, 75.5)
- moved D16 70.9 mm to (63.4, 73.8), turned to 0 degrees
- moved C78 68.1 mm to (97.0, 78.9)
- moved C68 67.4 mm to (97.0, 68.8), turned to 0 degrees
- moved C44 66.5 mm to (91.0, 65.5), turned to 0 degrees
- moved C81 62.3 mm to (97.0, 82.2)
- moved C62 60.5 mm to (91.0, 85.6), turned to 0 degrees
- moved C72 60.5 mm to (97.0, 72.2), turned to 0 degrees
- moved D5 57.6 mm to (46.5, 93.6)
- moved D6 57.6 mm to (46.5, 100.2)
- moved D7 57.6 mm to (46.5, 106.9)
- moved D12 57.5 mm to (55.0, 93.6)
- moved D9 57.5 mm to (55.0, 73.8)
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Connections:
- C29 pad 1: +3V3 -> +5V
- C30 pad 1: +3V3 -> +5V
- C31 pad 1: +3V3 -> +5V
- C32 pad 1: +3V3 -> +5V
- C33 pad 1: +3V3 -> +5V
- C34 pad 1: +3V3 -> +5V
- C35 pad 1: +3V3 -> +5V
- C36 pad 1: +3V3 -> +5V
- C47 pad 1: +3V3 -> +5V
- C48 pad 1: +3V3 -> +5V
- C49 pad 1: +3V3 -> +5V
- C50 pad 1: +3V3 -> +5V
- C51 pad 1: +3V3 -> +5V
- C52 pad 1: +3V3 -> +5V
- C53 pad 1: +3V3 -> +5V
- C54 pad 1: +3V3 -> +5V
- C55 pad 1: +3V3 -> +5V
- C56 pad 1: +3V3 -> +5V
- C57 pad 1: +3V3 -> +5V
- C58 pad 1: +3V3 -> +5V
- C59 pad 1: +3V3 -> +5V
- C60 pad 1: +3V3 -> +5V
- C61 pad 1: +3V3 -> +5V
- C62 pad 1: +3V3 -> +5V
- C63 pad 1: +3V3 -> +5V
- C64 pad 1: +3V3 -> +5V
- C65 pad 1: +3V3 -> +5V
- C66 pad 1: +3V3 -> +5V
- C67 pad 1: +3V3 -> +5V
- C68 pad 1: +3V3 -> +5V
- C69 pad 1: +3V3 -> +5V
- C71 pad 1: +3V3 -> +5V
- C72 pad 1: +3V3 -> +5V
- C73 pad 1: +3V3 -> +5V
- C74 pad 1: +3V3 -> +5V
- C75 pad 1: +3V3 -> +5V
- C76 pad 1: +3V3 -> +5V
- C77 pad 1: +3V3 -> +5V
- C78 pad 1: +3V3 -> +5V
- C79 pad 1: +3V3 -> +5V
- C80 pad 1: +3V3 -> +5V
- C81 pad 1: +3V3 -> +5V
- C82 pad 1: +3V3 -> +5V
- C83 pad 1: +3V3 -> +5V
- C84 pad 1: +3V3 -> +5V
- C85 pad 1: +3V3 -> +5V
- C86 pad 1: +3V3 -> +5V
- C88 pad 1: +3V3 -> +5V
- C89 pad 1: +3V3 -> +5V
- C91 pad 1: +3V3 -> +5V
- C92 pad 1: +3V3 -> +5V
- C94 pad 1: +3V3 -> +5V
- C95 pad 1: +3V3 -> +5V
- D13 pad 3: +3V3 -> +5V
- D14 pad 3: +3V3 -> +5V
- D15 pad 3: +3V3 -> +5V
- D16 pad 3: +3V3 -> +5V
- D17 pad 3: +3V3 -> +5V
- D18 pad 3: +3V3 -> +5V
- D19 pad 3: +3V3 -> +5V
- D20 pad 3: +3V3 -> +5V
- D21 pad 3: +3V3 -> +5V
- D22 pad 3: +3V3 -> +5V
- D23 pad 3: +3V3 -> +5V
- D24 pad 3: +3V3 -> +5V
- D25 pad 3: +3V3 -> +5V
- D300 pad 2: +3V3 -> +5V
- D301 pad 2: +3V3 -> +5V
- D302 pad 2: +3V3 -> +5V
- D303 pad 2: +3V3 -> +5V
- D304 pad 2: +3V3 -> +5V
- D305 pad 2: +3V3 -> +5V
- D306 pad 2: +3V3 -> +5V
- D307 pad 2: +3V3 -> +5V
- D37 pad 2: /LED Array 2/sk_pin1 -> /LED Array 1/sk_output_pin
- D37 pad 3: +3V3 -> +5V
- D38 pad 2: /LED Array 2/sk_pin2 -> Net-(D37-DOUT)
- D38 pad 3: +3V3 -> +5V
- D39 pad 2: /LED Array 1/sk_output_pin -> Net-(D38-DOUT)
- D40 pad 2: Net-(D37-DOUT) -> Net-(D39-DOUT)
- D40 pad 3: +3V3 -> +5V
- D41 pad 2: Net-(D38-DOUT) -> Net-(D40-DOUT)
- D41 pad 3: +3V3 -> +5V
- D42 pad 2: Net-(D39-DOUT) -> Net-(D41-DOUT)
- D43 pad 2: Net-(D40-DOUT) -> Net-(D42-DOUT)
- D43 pad 3: +3V3 -> +5V
- D44 pad 2: Net-(D41-DOUT) -> Net-(D43-DOUT)
- D44 pad 3: +3V3 -> +5V
- D44 pad 4: /LED Array 2/sk_output_pin -> Net-(D44-DOUT)
- D45 pad 2: Net-(D42-DOUT) -> Net-(D44-DOUT)
- D46 pad 2: Net-(D43-DOUT) -> Net-(D45-DOUT)
- D46 pad 3: +3V3 -> +5V
- D47 pad 2: Net-(D45-DOUT) -> Net-(D46-DOUT)
- D48 pad 2: Net-(D46-DOUT) -> Net-(D47-DOUT)
- D48 pad 3: +3V3 -> +5V
- D48 pad 4: Net-(D48-DOUT) -> /LED Array 2/sk_pin1
- D49 pad 2: Net-(D47-DOUT) -> /LED Array 2/sk_pin1
- D50 pad 2: Net-(D48-DOUT) -> Net-(D49-DOUT)
- D50 pad 3: +3V3 -> +5V
- D51 pad 2: Net-(D49-DOUT) -> Net-(D50-DOUT)
- D52 pad 2: Net-(D50-DOUT) -> Net-(D51-DOUT)
- D52 pad 3: +3V3 -> +5V
- D53 pad 2: Net-(D51-DOUT) -> Net-(D52-DOUT)
- D54 pad 2: Net-(D52-DOUT) -> Net-(D53-DOUT)
- D54 pad 3: +3V3 -> +5V
- D55 pad 2: Net-(D53-DOUT) -> Net-(D54-DOUT)
- D56 pad 2: Net-(D54-DOUT) -> Net-(D55-DOUT)
- D56 pad 3: +3V3 -> +5V
- D57 pad 2: Net-(D55-DOUT) -> Net-(D56-DOUT)
- D58 pad 2: Net-(D56-DOUT) -> Net-(D57-DOUT)
- D58 pad 3: +3V3 -> +5V
- D59 pad 2: Net-(D57-DOUT) -> Net-(D58-DOUT)
- D60 pad 2: Net-(D58-DOUT) -> Net-(D59-DOUT)
- D60 pad 3: +3V3 -> +5V
- D61 pad 2: Net-(D59-DOUT) -> Net-(D60-DOUT)
- D61 pad 4: Net-(D61-DOUT) -> /LED Array 2/sk_pin2
- D62 pad 2: Net-(D60-DOUT) -> /LED Array 2/sk_pin2
- D62 pad 3: +3V3 -> +5V
- D63 pad 2: Net-(D61-DOUT) -> Net-(D62-DOUT)
- D63 pad 4: /LED Array 2/sk_pin1 -> Net-(D63-DOUT)
- D64 pad 2: Net-(D62-DOUT) -> Net-(D63-DOUT)
- D64 pad 3: +3V3 -> +5V
- D64 pad 4: /LED Array 2/sk_pin2 -> /LED Array 2/sk_output_pin
- D65 pad 2: /LED Array 3/sk_pin1 -> /LED Array 2/sk_output_pin
- D65 pad 3: +3V3 -> +5V
- D66 pad 2: /LED Array 3/sk_pin2 -> Net-(D65-DOUT)
- D66 pad 3: +3V3 -> +5V
- D67 pad 2: /LED Array 2/sk_output_pin -> Net-(D66-DOUT)
- D68 pad 2: Net-(D65-DOUT) -> Net-(D67-DOUT)
- D68 pad 3: +3V3 -> +5V
- D69 pad 2: Net-(D66-DOUT) -> Net-(D68-DOUT)
- D69 pad 3: +3V3 -> +5V
- D70 pad 2: Net-(D67-DOUT) -> Net-(D69-DOUT)
- D71 pad 2: Net-(D68-DOUT) -> Net-(D70-DOUT)
- D71 pad 3: +3V3 -> +5V
- D72 pad 2: Net-(D69-DOUT) -> Net-(D71-DOUT)
- D72 pad 3: +3V3 -> +5V
- D72 pad 4: /LED Array 3/sk_output_pin -> Net-(D72-DOUT)
- D73 pad 2: Net-(D70-DOUT) -> Net-(D72-DOUT)
- D74 pad 2: Net-(D71-DOUT) -> Net-(D73-DOUT)
- D74 pad 3: +3V3 -> +5V
- D75 pad 2: Net-(D73-DOUT) -> Net-(D74-DOUT)
- D76 pad 2: Net-(D74-DOUT) -> Net-(D75-DOUT)
- D76 pad 3: +3V3 -> +5V
- D76 pad 4: Net-(D76-DOUT) -> /LED Array 3/sk_pin1
- D77 pad 2: Net-(D75-DOUT) -> /LED Array 3/sk_pin1
- D78 pad 2: Net-(D76-DOUT) -> Net-(D77-DOUT)
- D78 pad 3: +3V3 -> +5V
- D79 pad 2: Net-(D77-DOUT) -> Net-(D78-DOUT)
- D80 pad 2: Net-(D78-DOUT) -> Net-(D79-DOUT)
- D80 pad 3: +3V3 -> +5V
- D81 pad 2: Net-(D79-DOUT) -> Net-(D80-DOUT)
- D82 pad 2: Net-(D80-DOUT) -> Net-(D81-DOUT)
- D82 pad 3: +3V3 -> +5V
- D83 pad 2: Net-(D81-DOUT) -> Net-(D82-DOUT)
- D84 pad 2: Net-(D82-DOUT) -> Net-(D83-DOUT)
- D84 pad 3: +3V3 -> +5V
- D85 pad 2: Net-(D83-DOUT) -> Net-(D84-DOUT)
- D86 pad 2: Net-(D84-DOUT) -> Net-(D85-DOUT)
- D86 pad 3: +3V3 -> +5V
- D87 pad 2: Net-(D85-DOUT) -> Net-(D86-DOUT)
- D88 pad 2: Net-(D86-DOUT) -> Net-(D87-DOUT)
- D88 pad 3: +3V3 -> +5V
- D89 pad 2: Net-(D87-DOUT) -> Net-(D88-DOUT)
- D89 pad 4: Net-(D89-DOUT) -> /LED Array 3/sk_pin2
- D90 pad 2: Net-(D88-DOUT) -> /LED Array 3/sk_pin2
- D90 pad 3: +3V3 -> +5V
- D91 pad 2: Net-(D89-DOUT) -> Net-(D90-DOUT)
- D91 pad 4: /LED Array 3/sk_pin1 -> Net-(D91-DOUT)
- D92 pad 2: Net-(D90-DOUT) -> Net-(D91-DOUT)
- D92 pad 3: +3V3 -> +5V
- D92 pad 4: /LED Array 3/sk_pin2 -> /LED Array 3/sk_output_pin
Routing:
- net GND: track 1712.3 -> 0.00 mm, vias 5 -> 0
- net +3V3: track 1078.1 -> 0.00 mm, vias 18 -> 0
- net +5V: track 981.3 -> 0.00 mm, vias 17 -> 0
- net /LED Array 1/sk_output_pin: track 111.6 -> 0.00 mm, vias 2 -> 0
- net +12V: track 99.9 -> 0.00 mm
- net /LED Array 2/sk_output_pin: track 72.7 -> 0.00 mm, vias 2 -> 0
- net Net-(D20-DOUT): track 71.2 -> 0.00 mm, vias 2 -> 0
- net /LED Array 3/sk_pin1: track 68.8 -> 0.00 mm, vias 2 -> 0
- net /LED Array 2/sk_pin2: track 61.0 -> 0.00 mm, vias 2 -> 0
- net Net-(D51-DOUT): track 60.0 -> 0.00 mm, vias 2 -> 0
- net /LED Array 3/sk_pin2: track 58.8 -> 0.00 mm, vias 2 -> 0
- net /LED Array 2/sk_pin1: track 57.6 -> 0.00 mm, vias 2 -> 0
- net Net-(U1-VFB): track 50.5 -> 0.00 mm, vias 2 -> 0
- net Net-(D16-DOUT): track 48.2 -> 0.00 mm
- net Net-(D88-DOUT): track 48.1 -> 0.00 mm, vias 4 -> 0
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- removed copper zone on F.Cu, net GND

Commit message: Placed so many capacitors, dear lord
Parts:
- moved D307 204.7 mm to (34.1, 146.1), turned to 90 degrees
- moved D306 199.6 mm to (34.1, 133.2), turned to 90 degrees
- moved C36 195.6 mm to (36.9, 146.1), turned to 90 degrees
- moved D305 194.9 mm to (34.1, 120.3), turned to 90 degrees
- moved C35 190.7 mm to (36.8, 133.3), turned to 90 degrees
- moved D304 190.6 mm to (34.1, 107.4), turned to 90 degrees
- moved D303 186.7 mm to (34.1, 94.5), turned to 90 degrees
- moved C34 186.0 mm to (36.9, 120.3), turned to 90 degrees
- moved D302 183.3 mm to (34.1, 81.7), turned to 90 degrees
- moved C33 181.7 mm to (36.9, 107.3), turned to 90 degrees
- moved D301 180.4 mm to (34.1, 68.8), turned to 90 degrees
- moved D300 177.9 mm to (34.1, 55.9), turned to 90 degrees
- moved C32 177.9 mm to (37.0, 94.5), turned to 90 degrees
- moved C31 174.6 mm to (36.8, 81.6), turned to 90 degrees
- moved C30 171.8 mm to (36.8, 68.8), turned to 90 degrees
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