File: TeamSignFront/TeamSign.kicad_pcb (KiCad board)
At the start: 2 copper layers, 240 x 145 mm, 4 parts

Commit message: Update BOM + team sign PCB to not have diffuser issue.
Routing:
- removed copper zone on B.Cu, net (none)
Other:
- board text added: "JLCJLCJLCJLC"
- board text removed: "interior face pls"
- board text removed: "locked"
Changed lines of the file:
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@@
   (paper "A4")
   (title_block
-    (title "Team Timer w/ Stacklight")
-    (date "2023-05-10")
-    (rev "0.2b")
+    (title "Team Timer Diffuser")
+    (date "2023-05-22")
+    (rev "0.3b")
     (company "Garden State Combat Robotics League")
     (comment 3 "Kim Chase")
@@
   (gr_arc locked (start 30 160) (mid 26.464466 158.535534) (end 25 155)
     (stroke (width 0.1) (type default)) (layer "Edge.Cuts"))
-  (gr_text "interior face pls" (at 118.491 39.37) (layer "B.SilkS")
+  (gr_text "JLCJLCJLCJLC" (at 210.82 156.21) (layer "B.SilkS")
     (effects (font (size 1.5 1.5) (thickness 0.3) bold) (justify left bottom mirror))
   )
@@
       )
     )
-  )
-  (gr_text locked "888" (at 26 162.7) (layer "F.CrtYd")
-    (effects (font (face "DSEG7 Classic Mini") (size 70 70) (thickness 0.3) bold) (justify left bottom))
-    (render_cache "888" 0
-      (polygon
-        (pts
-          (xy 39.352756 143.636357)          (xy 35.745289 140.148569)          (xy 35.745289 103.526796)          (xy 38.292742 103.526796)
-          (xy 39.72889 104.945847)          (xy 46.003489 111.134961)          (xy 46.003489 137.088206)
-        )
-      )
-      (polygon
-        (pts
-          (xy 39.72889 97.081228)          (xy 38.292742 98.500279)          (xy 35.745289 98.500279)          (xy 35.745289 61.998185)
-          (xy 39.352756 58.390718)          (xy 46.003489 64.938869)          (xy 46.003489 90.892114)
-        )
-      )
-      (polygon
-        (pts
-          (xy 42.908932 54.834542)          (xy 46.39672 51.227076)          (xy 87.053384 51.227076)          (xy 90.541172 54.834542)
-          (xy 83.993021 61.485275)          (xy 49.47418 61.485275)
-        )
-      )
-      (polygon
-        (pts
-          (xy 85.463363 95.935729)          (xy 90.541172 101.013538)          (xy 85.463363 106.091346)          (xy 47.986741 106.091346)
-          (xy 42.908932 101.013538)          (xy 47.986741 95.935729)
-        )
-      )
-      (polygon
-        (pts
-          (xy 94.097348 58.390718)          (xy 97.704815 61.878506)          (xy 97.704815 98.500279)          (xy 95.157362 98.500279)
-          (xy 93.721214 97.081228)          (xy 87.446615 90.892114)          (xy 87.446615 64.938869)
-        )
-      )
-      (polygon
-        (pts
-          (xy 90.541172 147.192533)          (xy 87.053384 150.8)          (xy 46.39672 150.8)          (xy 42.908932 147.192533)
-          (xy 49.47418 140.5418)          (xy 83.993021 140.5418)
-        )
-      )
-      (polygon
-        (pts
-          (xy 93.704117 104.945847)          (xy 95.157362 103.526796)          (xy 97.704815 103.526796)          (xy 97.704815 140.148569)
-          (xy 94.097348 143.636357)          (xy 87.446615 137.088206)          (xy 87.446615 111.237543)
-        )
-      )
-      (polygon
-        (pts
-          (xy 119.298325 143.636357)          (xy 115.690858 140.148569)          (xy 115.690858 103.526796)          (xy 118.238311 103.526796)
-          (xy 119.674459 104.945847)          (xy 125.949057 111.134961)          (xy 125.949057 137.088206)
-        )
-      )
-      (polygon
-        (pts
-          (xy 119.674459 97.081228)          (xy 118.238311 98.500279)          (xy 115.690858 98.500279)          (xy 115.690858 61.998185)
-          (xy 119.298325 58.390718)          (xy 125.949057 64.938869)          (xy 125.949057 90.892114)
-        )
-      )
-      (polygon
-        (pts
-          (xy 122.854501 54.834542)          (xy 126.342288 51.227076)          (xy 166.998953 51.227076)          (xy 170.486741 54.834542)
-          (xy 163.93859 61.485275)          (xy 129.419748 61.485275)
-        )
-      )
-      (polygon
-        (pts
-          (xy 165.408932 95.935729)          (xy 170.486741 101.013538)          (xy 165.408932 106.091346)          (xy 127.932309 106.091346)
-          (xy 122.854501 101.013538)          (xy 127.932309 95.935729)
-        )
-      )
-      (polygon
-        (pts
-          (xy 174.042916 58.390718)          (xy 177.650383 61.878506)          (xy 177.650383 98.500279)          (xy 175.10293 98.500279)
-          (xy 173.666782 97.081228)          (xy 167.392184 90.892114)          (xy 167.392184 64.938869)
-        )
-      )
-      (polygon
-        (pts
-          (xy 170.486741 147.192533)          (xy 166.998953 150.8)          (xy 126.342288 150.8)          (xy 122.854501 147.192533)
-          (xy 129.419748 140.5418)          (xy 163.93859 140.5418)
-        )
-      )
-      (polygon
-        (pts
-          (xy 173.649685 104.945847)          (xy 175.10293 103.526796)          (xy 177.650383 103.526796)          (xy 177.650383 140.148569)
-          (xy 174.042916 143.636357)          (xy 167.392184 137.088206)          (xy 167.392184 111.237543)
-        )
-      )
-      (polygon
-        (pts
-          (xy 199.243893 143.636357)          (xy 195.636427 140.148569)          (xy 195.636427 103.526796)          (xy 198.183879 103.526796)
-          (xy 199.620027 104.945847)          (xy 205.894626 111.134961)          (xy 205.894626 137.088206)
-        )
-      )
-      (polygon
-        (pts
-          (xy 199.620027 97.081228)          (xy 198.183879 98.500279)          (xy 195.636427 98.500279)          (xy 195.636427 61.998185)
-          (xy 199.243893 58.390718)          (xy 205.894626 64.938869)          (xy 205.894626 90.892114)
-        )
-      )
-      (polygon
-        (pts
-          (xy 202.800069 54.834542)          (xy 206.287857 51.227076)          (xy 246.944521 51.227076)          (xy 250.432309 54.834542)
-          (xy 243.884159 61.485275)          (xy 209.365317 61.485275)
-        )
-      )
-      (polygon
-        (pts
-          (xy 245.354501 95.935729)          (xy 250.432309 101.013538)          (xy 245.354501 106.091346)          (xy 207.877878 106.091346)
-          (xy 202.800069 101.013538)          (xy 207.877878 95.935729)
-        )
-      )
-      (polygon
-        (pts
-          (xy 253.988485 58.390718)          (xy 257.595952 61.878506)          (xy 257.595952 98.500279)          (xy 255.048499 98.500279)
-          (xy 253.612351 97.081228)          (xy 247.337752 90.892114)          (xy 247.337752 64.938869)
-        )
-      )
-      (polygon
-        (pts
-          (xy 250.432309 147.192533)          (xy 246.944521 150.8)          (xy 206.287857 150.8)          (xy 202.800069 147.192533)
-          (xy 209.365317 140.5418)          (xy 243.884159 140.5418)
-        )
-      )
-      (polygon
-        (pts
-          (xy 253.595254 104.945847)          (xy 255.048499 103.526796)          (xy 257.595952 103.526796)          (xy 257.595952 140.148569)
-          (xy 253.988485 143.636357)          (xy 247.337752 137.088206)          (xy 247.337752 111.237543)
-        )
-      )
-    )
-  )
-  (zone (net 0) (net_name "") (layer "B.Cu") (hatch edge 0.5)
-    (priority 1)
-    (connect_pads (clearance 0.5))
-    (min_thickness 0.25) (filled_areas_thickness no)
-    (fill yes (thermal_gap 0.4) (thermal_bridge_width 0.4) (island_removal_mode 1) (island_area_min 10))
-    (polygon
-      (pts
-        (xy 20.32 5.5)
-        (xy 281.94 5.08)
-        (xy 281.94 162.56)
-        (xy 20.32 162.56)
-      )
-    )
