File: ArenaController/ArenaController.kicad_pcb (KiCad board)
At the start: 2 copper layers, 80 x 90 mm, 26 parts, among them J1 RJ45, J2 RJ45, J4 RJ45, J5 RJ45, J6 RJ45, J9 Barrel_Jack_MountingPin, Q1 FS3400, Q2 FS3400, Q3 FS3400, Q4 FS3400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

Commit message: Added Littelfuse TVS to the schematic.
Parts:
- added T1: ~, Package_TO_SOT_SMD:SOT-143_Handsoldering, F.Cu at (106.2, 60.5)
Routing:
- net +12V: track 122.3 -> 125.0 mm
- net GND: vias 97 -> 96
Changed lines of the file:
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@@
   (net 67 "unconnected-(U3-RTC_GPIO5{slash}ADC1_7{slash}GPIO35-Pad25)")
   (net 68 "unconnected-(J9-MountPin-Pad3)")
+  (net 69 "unconnected-(T1-IO1-Pad2)")
+  (net 70 "unconnected-(T1-IO2-Pad3)")
   (footprint "Package_TO_SOT_SMD:SOT-23" (layer "F.Cu")
     (at 135.2804 90.8812 90)
@@
       (net 6 "GND") (pintype "passive"))
   )
+  (footprint "Package_TO_SOT_SMD:SOT-143_Handsoldering" (layer "F.Cu")
+    (at 106.172 60.452)
+    (descr "SOT-143 Handsoldering https://www.nxp.com/docs/en/package-information/SOT143B.pdf")
+    (tags "SOT-143 Handsoldering")
+    (property "LCSC" "https://www.lcsc.com/product-detail/ESD-Protection-Devices_Littelfuse-SR70-02CTG_C1973334.html")
+    (property "Sheetfile" "ArenaController.kicad_sch")
+    (property "Sheetname" "")
+    (property "ki_description" "Littelfuse 12V TVS")
+    (attr smd)
+    (fp_text reference "T1" (at -0.02 -2.38) (layer "F.SilkS")
+        (effects (font (size 1 1) (thickness 0.15)))
+    )
+    (fp_text value "~" (at -0.02 2.48) (layer "F.Fab")
+        (effects (font (size 1 1) (thickness 0.15)))
+    )
+    (fp_text user "${REFERENCE}" (at 0 0 90) (layer "F.Fab")
+        (effects (font (size 0.5 0.5) (thickness 0.075)))
+    )
+    (fp_line (start -0.65 1.56) (end 0.65 1.56)
+      (stroke (width 0.12) (type solid)) (layer "F.SilkS"))
+    (fp_line (start 0.65 -1.56) (end -2.35 -1.56)
+      (stroke (width 0.12) (type solid)) (layer "F.SilkS"))
+    (fp_line (start -2.6 1.7) (end -2.6 -1.7)
+      (stroke (width 0.05) (type solid)) (layer "F.CrtYd"))
+    (fp_line (start -2.6 1.7) (end 2.6 1.7)
+      (stroke (width 0.05) (type solid)) (layer "F.CrtYd"))
+    (fp_line (start 2.6 -1.7) (end -2.6 -1.7)
+      (stroke (width 0.05) (type solid)) (layer "F.CrtYd"))
+    (fp_line (start 2.6 -1.7) (end 2.6 1.7)
+      (stroke (width 0.05) (type solid)) (layer "F.CrtYd"))
+    (fp_line (start -0.65 -0.95) (end -0.15 -1.45)
+      (stroke (width 0.1) (type solid)) (layer "F.Fab"))
+    (fp_line (start -0.65 1.45) (end -0.65 -0.95)
+      (stroke (width 0.1) (type solid)) (layer "F.Fab"))
+    (fp_line (start -0.15 -1.45) (end 0.65 -1.45)
+      (stroke (width 0.1) (type solid)) (layer "F.Fab"))
+    (fp_line (start 0.65 -1.45) (end 0.65 1.45)
+      (stroke (width 0.1) (type solid)) (layer "F.Fab"))
+    (fp_line (start 0.65 1.45) (end -0.65 1.45)
+      (stroke (width 0.1) (type solid)) (layer "F.Fab"))
+    (pad "1" smd rect (at -1.5 -0.75) (size 1.7 1) (layers "F.Cu" "F.Paste" "F.Mask")
+      (net 6 "GND") (pinfunction "GND") (pintype "input"))
+    (pad "2" smd rect (at -1.5 0.95) (size 1.7 0.6) (layers "F.Cu" "F.Paste" "F.Mask")
+      (net 69 "unconnected-(T1-IO1-Pad2)") (pinfunction "IO1") (pintype "input"))
+    (pad "3" smd rect (at 1.5 0.95) (size 1.7 0.6) (layers "F.Cu" "F.Paste" "F.Mask")
+      (net 70 "unconnected-(T1-IO2-Pad3)") (pinfunction "IO2") (pintype "input"))
+    (pad "4" smd rect (at 1.5 -0.95) (size 1.7 0.6) (layers "F.Cu" "F.Paste" "F.Mask")
+      (net 1 "+12V") (pinfunction "VCC") (pintype "input"))
+    (model "${KICAD6_3DMODEL_DIR}/Package_TO_SOT_SMD.3dshapes/SOT-143.wrl"
+      (offset (xyz 0 0 0))
+      (scale (xyz 1 1 1))
+      (rotate (xyz 0 0 0))
+    )
+  )
   (footprint "Inductor_SMD:L_1210_3225Metric_Pad1.42x2.65mm_HandSolder" (layer "F.Cu")
     (at 132.9944 52.5272 -90)
@@
   (segment (start 120.904 58.832) (end 160.018825 58.832) (width 1) (layer "F.Cu") (net 1))
   (segment (start 116.078 58.166) (end 120.238 58.166) (width 1) (layer "F.Cu") (net 1))
-  (segment (start 110.236 53.975) (end 110.236 62.865) (width 1) (layer "F.Cu") (net 1))
   (segment (start 129.794 55.372) (end 129.794 54.61) (width 0.6) (layer "F.Cu") (net 1))
+  (segment (start 110.236 59.309) (end 110.236 62.865) (width 1) (layer "F.Cu") (net 1))
   (segment (start 120.904 58.832) (end 120.904 54.3535) (width 1) (layer "F.Cu") (net 1))
   (segment (start 120.238 58.166) (end 120.904 58.832) (width 1) (layer "F.Cu") (net 1))
   (segment (start 128.524 53.34) (end 121.9175 53.34) (width 0.6) (layer "F.Cu") (net 1))
+  (segment (start 110.043 59.502) (end 107.672 59.502) (width 1) (layer "F.Cu") (net 1))
   (segment (start 110.236 62.865) (end 104.25 68.851) (width 1) (layer "F.Cu") (net 1))
   (segment (start 169.545 68.358175) (end 169.545 82.042) (width 1) (layer "F.Cu") (net 1))
+  (segment (start 110.236 53.975) (end 110.236 59.309) (width 1) (layer "F.Cu") (net 1))
+  (segment (start 110.236 59.309) (end 110.043 59.502) (width 1) (layer "F.Cu") (net 1))
   (segment (start 169.545 82.042) (end 167.542 84.045) (width 1) (layer "F.Cu") (net 1))
   (segment (start 111.887 53.975) (end 116.078 58.166) (width 1) (layer "F.Cu") (net 1))
@@
   (via (at 156.4132 61.976) (size 0.8) (drill 0.4) (layers "F.Cu" "B.Cu") (free) (net 6))
   (via (at 161.29 68.072) (size 0.8) (drill 0.4) (layers "F.Cu" "B.Cu") (free) (net 6))
-  (via (at 103.9876 96.4184) (size 0.8) (drill 0.4) (layers "F.Cu" "B.Cu") (free) (net 6))
   (via (at 106.4768 89.9668) (size 0.8) (drill 0.4) (layers "F.Cu" "B.Cu") (free) (net 6))
   (via (at 156.21 94.996) (size 0.8) (drill 0.4) (layers "F.Cu" "B.Cu") (free) (net 6))

Commit message: Update board to have less skullfscked routing and removed unused projects.
Parts:
- removed T1: ~, Package_TO_SOT_SMD:SOT-143_Handsoldering
- added D1: D_TVS, Diode_SMD:D_SOD-123F, F.Cu at (118.1, 52.7)
- moved C1 2.81 mm to (123.6, 52.6)
- moved U2 2.44 mm to (130.3, 52.8)
- moved C2 2.44 mm to (142.4, 52.4)
- moved L1 2.44 mm to (135.4, 52.5)
Connections:
- U3 pad 12: /T_B_Start -> /G_Start
- U3 pad 14: /G_Start -> /G_RST
- U3 pad 17: /G_End -> /G_Pause
- U3 pad 18: /T_B_End -> /G_End
- U3 pad 30: /G_RST -> unconnected-(U3-RTC_GPIO17/Touch7/ADC2_7/GPIO27-Pad30)
- U3 pad 31: /G_Pause -> unconnected-(U3-RTC_GPIO16/Touch6/HSPI_CLK/ADC2_6/GPIO14-Pad31)
- U3 pad 8: /Dis_serial_Rx -> /T_B_End
- U3 pad 9: /Dis_Serial_Tx -> /T_B_Start
Routing:
- net /G_Pause: track 66.4 -> 17.8 mm, vias 2 -> 0
- net /G_RST: track 60.9 -> 23.0 mm, vias 1 -> 0
- net /T_B_End: track 32.4 -> 19.3 mm, vias 1 -> 0
- net /G_End: track 22.2 -> 19.4 mm
- net +12V: track 125.0 -> 127.3 mm
- net /G_Start: track 19.9 -> 22.0 mm
- net /T_B_Start: track 20.2 -> 22.3 mm
- net /s_Green: track 95.6 -> 97.1 mm
- net +5V: track 38.7 -> 37.3 mm
- net /s_Horn: track 96.6 -> 97.5 mm, vias 1 -> 0
- net /s_Yellow: track 110.0 -> 109.2 mm
- net GND: vias 96 -> 98

Commit message: Added test points and 3D model for pin headers to the ESP32 footprint.
Parts:
- added TP1: TestPoint, TestPoint:TestPoint_Loop_D1.80mm_Drill1.0mm_Beaded, F.Cu at (105.1, 57.4)
- added TP2: TestPoint, TestPoint:TestPoint_Loop_D1.80mm_Drill1.0mm_Beaded, F.Cu at (106.0, 61.2)
- added TP3: TestPoint, TestPoint:TestPoint_Loop_D1.80mm_Drill1.0mm_Beaded, F.Cu at (148.4, 52.5)
- added TP4: TestPoint, TestPoint:TestPoint_Loop_D1.80mm_Drill1.0mm_Beaded, F.Cu at (151.2, 55.6)
Routing:
- net +5V: track 37.3 -> 44.3 mm
- net +12V: track 127.3 -> 133.9 mm
